File: Wisp.kicad_sch (KiCad schematic)
At the start: 12 parts, among them J1 USB4105-GF-A, J2 SM04B-GHS-TB, U1 ESP32-S3-MINI-1, U2 USBLC6-2SC6, U3 AP2112K-3.3TRG1, U4 TPS7A2033PYCJR

Commit message: Added components and wired EN button and GPIO
Parts:
- added S1: TS04-66-50-BK-160-SMT, TS04-66-50-BK-160-SMT:SW_TS04-66-50-BK-160-SMT, symbol TS04-66-50-BK-160-SMT:TS04-66-50-BK-160-SMT
Connections:
- net GND: now also S1.4
- net UWB_WAKE: now reaches U1.10 (IO6)
- net DIP_ID1: now reaches U1.11 (IO7)
- net DIP_ID2: now reaches U1.12 (IO8)
- net BTN_CAL: now reaches U1.13 (IO9)
- net UWB_CS: now reaches U1.14 (IO10)
- net UWB_MOSI: now reaches U1.15 (IO11)
- net USB_SCLK: now reaches U1.16 (IO12)
- net USB_MISO: now reaches U1.17 (IO13)
- net IO14: now reaches U1.18 (IO14)
- net IO15: now reaches U1.19 (IO15)
- net IO16: now reaches U1.20 (IO16)
- net FC_TX: now reaches U1.21 (IO17)
- net FC_RX: now reaches U1.22 (IO18)
- net LED_STATUS: now reaches U1.25 (IO21)
- net IO26: now reaches U1.26 (IO26)
- net IO47: now reaches U1.27 (IO47)
- net IO33: now reaches U1.28 (IO33)
- net IO34: now reaches U1.29 (IO34)
- net IO48: now reaches U1.30 (IO48)
- net IO35: now reaches U1.31 (IO35)
- net IO36: now reaches U1.32 (IO36)
- net IO37: now reaches U1.33 (IO37)
- net IO38: now reaches U1.34 (IO38)
- net IO39: now reaches U1.35 (IO39)
- net IO40: now reaches U1.36 (IO40)
- net IO41: now reaches U1.37 (IO41)
- net IO42: now reaches U1.38 (IO42)
- net TXD0: now reaches U1.39 (TXD0)
- net RXD0: now reaches U1.40 (RXD0)
- net EN: now reaches C3.2, R3.2, U1.45 (EN)
- net EN: now also S1.1
- net DIP_ROLE: now reaches U1.5 (IO1)
- net DIP_ID0: now reaches U1.6 (IO2)
- net UWB_IRQ: now reaches U1.8 (IO4)
- net UWB_RST: now reaches U1.9 (IO5)
- no-connect marks 2 -> 6

Commit message: Completed schematic; ERC remaining
Parts:
- added D1: LED, symbol Device:LED
- added H1: TL, symbol Mechanical:MountingHole_Pad_MP
- added H2: TR, symbol Mechanical:MountingHole_Pad_MP
- added H3: BR, symbol Mechanical:MountingHole_Pad_MP
- added H4: BL, symbol Mechanical:MountingHole_Pad_MP
- added J3, J4, J5: Conn_01x08_Pin, symbol Connector:Conn_01x08_Pin
- added R4: 100k, symbol Device:R_Small
- added R5, R6, R7: 10k, symbol Device:R_Small
- added S2: DS04-254-2-04BK-SMT-TR, DS04-254-2-04BK-SMT-TR:SW_DS04-254-2-04BK-SMT-TR, symbol DS04-254-2-04BK-SMT-TR:DS04-254-2-04BK-SMT-TR
- added S3: TS04-66-50-BK-160-SMT, TS04-66-50-BK-160-SMT:SW_TS04-66-50-BK-160-SMT, symbol TS04-66-50-BK-160-SMT:TS04-66-50-BK-160-SMT
- added TP1: UTX, symbol Connector:TestPoint
- added TP2: URX, symbol Connector:TestPoint
- added TP3: 5v, symbol Connector:TestPoint
- added TP4: 3v3, symbol Connector:TestPoint
- added TP5: 3v3U, symbol Connector:TestPoint
- added TP6: UMOSI, symbol Connector:TestPoint
- added TP7: UMISO, symbol Connector:TestPoint
- added TP8: USCLK, symbol Connector:TestPoint
- added TP9: UCS, symbol Connector:TestPoint
- added U5: DWM3000TR13, DWM3000TR13:XCVR_DWM3000TR13, symbol DWM3000TR13:DWM3000TR13
Connections:
- net +3V3: now also TP4.1
- net +5V: now also TP3.1
- net BTN_CAL: now also S3.1
- net DIP_ID0: now also S2.2A
- net DIP_ID1: now also S2.3A
- net DIP_ID2: now also S2.4A
- net DIP_ROLE: now also S2.1A
- net GND: now also D1.2 (A), H1.MP, H2.MP, H3.MP, H4.MP, R4.2, R6.2, R7.2, S2.1B, S2.2B, S2.3B, S2.4B, S3.4, U5.16 (VSS), U5.21 (VSS), U5.23 (VSS), U5.24 (VSS), U5.8 (VSS)
- net IO14: now also J3.8 (Pin_8)
- net IO15: now also J3.7 (Pin_7)
- net IO16: now also J3.6 (Pin_6)
- net IO26: now also J3.5 (Pin_5)
- net IO33: now also J3.4 (Pin_4)
- net IO34: now also J3.3 (Pin_3)
- net IO35: now also J3.2 (Pin_2)
- net IO36: now also J3.1 (Pin_1)
- net IO37: now also J4.1 (Pin_1)
- net IO38: now also J4.2 (Pin_2)
- net IO39: now also J4.3 (Pin_3)
- net IO40: now also J4.4 (Pin_4)
- net IO41: now also J4.5 (Pin_5)
- net IO42: now also J4.6 (Pin_6)
- net IO47: now also J4.7 (Pin_7)
- net IO48: now also J4.8 (Pin_8)
- net LED_STATUS: now also D1.1 (K)
- net UART_RX: now also TP2.1
- net UART_TX: now also TP1.1
- net USB_MISO: now also TP7.1, U5.19 (SPIMISO)
- net USB_SCLK: now also TP8.1, U5.20 (SPICLK)
- net UWB_CS: now also R5.1, TP9.1, U5.17 (~{SPICS})
- net UWB_IRQ: now also U5.22 (GPIO8/IRQ)
- net UWB_MOSI: now also TP6.1, U5.18 (SPIMOSI)
- net UWB_RST: now also U5.3 (~{RST})
- net UWB_WAKE: now also R4.1, U5.2 (WAKEUP)
- net +3V3_UWB renamed VDD3V3
- net VDD3V3: now also R5.2, TP5.1, U5.5 (VDD1), U5.6 (VDD3V3), U5.7 (VDD3V3)
- new net EXTON: U5.1 (EXTON)
- new net GPIO0/RXOKLED: J5.8 (Pin_8), U5.15 (GPIO0/RXOKLED)
- new net GPIO1/SFDLED: J5.7 (Pin_7), U5.14 (GPIO1/SFDLED)
- new net GPIO2/RXLED: J5.6 (Pin_6), U5.13 (GPIO2/RXLED)
- new net GPIO3/TXLED: J5.5 (Pin_5), U5.12 (GPIO3/TXLED)
- new net GPIO4: J5.4 (Pin_4), U5.11 (GPIO4)
- new net GPIO5/EXTTXE/SPIPOL: J5.3 (Pin_3), R6.1, U5.10 (GPIO5/EXTTXE/SPIPOL)
- new net GPIO6/EXTRXE/SPIPHA: J5.2 (Pin_2), R7.1, U5.9 (GPIO6/EXTRXE/SPIPHA)
- new net GPIO7/SYNC: J5.1 (Pin_1), U5.4 (GPIO7/SYNC)
Other:
- moved on the sheet: C1, J2

Commit message: Started PCB routing; Completed Schematic
Parts:
- removed J3, J4, J5: Conn_01x08_Pin, symbol Connector:Conn_01x08_Pin
- removed R6, R7: 10k, symbol Device:R_Small
- removed S1, S3: TS04-66-50-BK-160-SMT, TS04-66-50-BK-160-SMT:SW_TS04-66-50-BK-160-SMT, symbol TS04-66-50-BK-160-SMT:TS04-66-50-BK-160-SMT
- removed S2: DS04-254-2-04BK-SMT-TR, DS04-254-2-04BK-SMT-TR:SW_DS04-254-2-04BK-SMT-TR, symbol DS04-254-2-04BK-SMT-TR:DS04-254-2-04BK-SMT-TR
- added J3, J4: Conn_01x05_Pin, Connector_PinHeader_2.54mm:PinHeader_1x05_P2.54mm_Vertical_SMD_Pin1Right, symbol Connector:Conn_01x05_Pin
- added J5, J6: Conn_01x04_Pin, Connector_PinHeader_2.54mm:PinHeader_1x04_P2.54mm_Vertical_SMD_Pin1Right, symbol Connector:Conn_01x04_Pin
- added J9: Conn_02x04_Counter_Clockwise, Connector_PinHeader_2.00mm:PinHeader_2x04_P2.00mm_Vertical, symbol Connector_Generic:Conn_02x04_Counter_Clockwise
- added SW2, SW3: PTS810 SJM 250 SMTR LFS, PTS810_SJM_250_SMTR_LFS:PTS810_CNK, symbol PTS810_SJM_250_SMTR_LFS:PTS810_SJM_250_SMTR_LFS
- C1, C2, C3: footprint (none) -> Capacitor_SMD:C_0201_0603Metric
- D1: footprint (none) -> LED_SMD:LED_0603_1608Metric
- H1, H2, H3, H4: footprint (none) -> MountingHole:MountingHole_3.2mm_M3_Pad_Via
- J1: footprint USB4105-GF-A:GCT_USB4105-GF-A -> USB4105_GF_A:GCT_USB4105-GF-A
- J2: footprint SM04B-GHS-TB:JST_SM04B-GHS-TB -> SM04B_GHS_TB:JST_SM04B-GHS-TB
- R1, R2, R3, R4, R5: footprint (none) -> Resistor_SMD:R_0603_1608Metric
- TP1, TP2, TP3, TP4, TP5, TP6, TP7, TP8, TP9: footprint (none) -> TestPoint:TestPoint_Pad_1.0x1.0mm
- U2: footprint USBLC6-2SC6:SOT95P280X145-6N -> USBLC6_2SC6:SOT95P280X145-6N
- U4: footprint YCJ0004-C01-IPC_A -> TPS7A2033PYCJR:TPS7A2033PYCJR
Connections:
- net UART_RX is gone; now on net FC_RX: J2.3, TP2.1
- net UART_TX is gone; now on net FC_TX: J2.2, TP1.1
- net BTN_CAL: now also SW3.1
- net DIP_ID0: now also J9.3 (Pin_3)
- net DIP_ID1: now also J9.5 (Pin_5)
- net DIP_ID2: now also J9.7 (Pin_7)
- net DIP_ROLE: now also J9.1 (Pin_1)
- net EN: now also SW2.1
- net GND: now also J9.2 (Pin_2), J9.4 (Pin_4), J9.6 (Pin_6), J9.8 (Pin_8), SW2.4, SW3.4
- net IO14: now also J4.3 (Pin_3)
- net IO15: now also J4.2 (Pin_2)
- net IO16: now also J4.1 (Pin_1)
- net IO26: now also J3.5 (Pin_5)
- net IO33: now also J3.4 (Pin_4)
- net IO34: now also J3.3 (Pin_3)
- net IO35: now also J3.2 (Pin_2)
- net IO36: now also J3.1 (Pin_1)
- net IO37: now also J5.1 (Pin_1)
- net IO38: now also J5.2 (Pin_2)
- net IO39: now also J5.3 (Pin_3)
- net IO40: now also J5.4 (Pin_4)
- net IO41: now also J6.1 (Pin_1)
- net IO42: now also J6.2 (Pin_2)
- net IO47: now also J6.3 (Pin_3)
- net IO48: now also J6.4 (Pin_4)
- net EXTON: no longer names the net of U5.1 (EXTON)
- net GPIO0/RXOKLED: no longer names the net of U5.15 (GPIO0/RXOKLED)
- net GPIO1/SFDLED: no longer names the net of U5.14 (GPIO1/SFDLED)
- net GPIO2/RXLED: no longer names the net of U5.13 (GPIO2/RXLED)
- net GPIO3/TXLED: no longer names the net of U5.12 (GPIO3/TXLED)
- net GPIO4: no longer names the net of U5.11 (GPIO4)
- net GPIO5/EXTTXE/SPIPOL: no longer names the net of U5.10 (GPIO5/EXTTXE/SPIPOL)
- net GPIO6/EXTRXE/SPIPHA: no longer names the net of U5.9 (GPIO6/EXTRXE/SPIPHA)
- net GPIO7/SYNC: no longer names the net of U5.4 (GPIO7/SYNC)
- net RXD0: no longer names the net of U1.40 (RXD0)
- net TXD0: no longer names the net of U1.39 (TXD0)
- net USB_MISO renamed UWB_MISO
- net USB_SCLK renamed UWB_SCLK
- no-connect marks 6 -> 23

Commit message: Completed V1.0
Parts:
- removed J3, J4: Conn_01x05_Pin, Connector_PinHeader_2.54mm:PinHeader_1x05_P2.54mm_Vertical_SMD_Pin1Right, symbol Connector:Conn_01x05_Pin
- removed J5: Conn_01x04_Pin, Connector_PinHeader_2.54mm:PinHeader_1x04_P2.54mm_Vertical_SMD_Pin1Right, symbol Connector:Conn_01x04_Pin
Connections:
- net IO14: no longer names the net of U1.18 (IO14)
- net IO15: no longer names the net of U1.19 (IO15)
- net IO16: no longer names the net of U1.20 (IO16)
- net IO26: no longer names the net of U1.26 (IO26)
- net IO33: no longer names the net of U1.28 (IO33)
- net IO34: no longer names the net of U1.29 (IO34)
- net IO35: no longer names the net of U1.31 (IO35)
- net IO36: no longer names the net of U1.32 (IO36)
- net IO37: no longer names the net of U1.33 (IO37)
- net IO38: no longer names the net of U1.34 (IO38)
- net IO39: no longer names the net of U1.35 (IO39)
- net IO40: no longer names the net of U1.36 (IO40)
- no-connect marks 23 -> 33

Commit message: Fixed bugs
Parts:
- removed U4: TPS7A2033PYCJR, TPS7A2033PYCJR:TPS7A2033PYCJR, symbol TPS7A2033PYCJR:TPS7A2033PYCJR
- added C4, C6: 1uF, Capacitor_SMD:C_0603_1608Metric, symbol Device:C_Small
- added C5: 10uF, Capacitor_SMD:C_0603_1608Metric, symbol Device:C_Small
- added U4: TPS7A2033PDBVR, TPS7A2033PDBVR:SOT95P280X145-5N, symbol TPS7A2033PDBVR:TPS7A2033PDBVR
- C1: footprint Capacitor_SMD:C_0201_0603Metric -> Capacitor_SMD:C_0603_1608Metric
- C2: value 22u -> 22uF; footprint Capacitor_SMD:C_0201_0603Metric -> Capacitor_SMD:C_0603_1608Metric
- C3: value 1u -> 1uF; footprint Capacitor_SMD:C_0201_0603Metric -> Capacitor_SMD:C_0603_1608Metric
- renumbered TP1 to T1
Connections:
- net +3V3: now also C6.1
- net +5V: now also U4.1 (IN), U4.3 (EN)
- net GND: now also D1.1 (K), C4.2, C5.2, C6.2, U4.2 (GND); no longer D1.2 (A)
- net LED_STATUS: now also D1.2 (A); no longer D1.1 (K)
- net VDD3V3: now also C4.1, C5.1, U4.5 (OUT)
Other:
- moved on the sheet: D1, J6

Commit message: Organized the schematic into sections
Other:
- note added: "Connectors/Test points"
- note added: "ESP32S3/UWB Module"
- note added: "Power regulators"
- note added: "Switches"
- note added: "USB-C and ESD"
- moved on the sheet: C1, C2, C3, C4, C5, C6, D1, H1, H2, H3, H4, J1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
